File: Electronics/TIA/_restore_backup_2026-05-16T12-51-38-184/TIA.kicad_sch (KiCad schematic)
At the start: 4 parts

Commit message: Create a robust TIA design following the requirements
Parts:
- removed V3: VPULSE, symbol Simulation_SPICE:VPULSE
Connections:
- net +5V renamed +15V
- net -5V renamed -15V
Other:
- removed sheet OPA859
- removed sheet OPA859 1G
