File: Electronics/ULCA/Different topology.kicad_sch (KiCad schematic)
At the start: 12 parts, among them U5 ${SIM.PARAMS}, U6 ${SIM.PARAMS}

Commit message: Create an okayish tunned ULCA
Parts:
- removed C5: 1p, symbol Device:C
- removed C6, C7, C8: 100f, symbol Device:C
- removed I3: ISIN, symbol Simulation_SPICE:ISIN
- removed R7: 1G, symbol Device:R
- removed R8, R9: 1M, symbol Device:R
- removed U5, U6: ${SIM.PARAMS}, symbol Simulation_SPICE:OPAMP
- removed V5, V6: 50V, symbol Simulation_SPICE:VDC
- added C10, C11, C12: 50f, symbol Device:C
- added C13: 10p, symbol Device:C
- added C9: 1p, symbol Device:C
- added I4: ISIN, symbol Simulation_SPICE:ISIN
- added R10, R12: 10M, symbol Device:R
- added R11: 10, symbol Device:R
- added U9: ${SIM.PARAMS}, symbol Simulation_SPICE:OPAMP
- added V7, V8: 50V, symbol Simulation_SPICE:VDC
Connections:
- net +50V: now also U9.3 (V+), V7.1
- net -50V: now also U9.4 (V-), V8.2
- net 0: now also C11.1, C9.2, I4.2, R11.2, U9.1 (+), V7.2, V8.1
- net VIN: now also C10.1, C9.1, I4.1, R10.1, U9.2 (-)
- net VOUT: now also C10.2, C11.2, C12.1, C12.2, C13.1, C13.2, R10.2, R11.1, R12.1, R12.2, U9.5
Other:
- note added: "This one is supprisingly good. But the op amp gain and feedback capacitance are unrealistic."
- note removed: "It's stable.r But the gain is too high. And the bandwidth is too small. Probably it can be improved with lower gain."
