File: Electronics/Peculiar/From OPA380.kicad_sch (KiCad schematic)
At the start: 12 parts, among them U2 ${SIM.PARAMS}, U3 ${SIM.PARAMS}

Commit message: Create a great design using OPA858 and OPA162
Parts:
- renumbered C3 to C1, C1 to C2, C2 to C3, R2 to R1, R3 to R2, R1 to R3, U2 to U1, U3 to U2
Changed lines of the file:
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@@
 		(dnp no)
 		(fields_autoplaced yes)
-		(property "Reference" "#PWR012"
+		(property "Reference" "#PWR010"
 			(at 167.64 120.65 0)
 			(hide yes)
@@
 			(project "Peculiar"
 				(path "/db27cf5d-1015-467f-a739-ab2eb7f0a1b5/f65afffd-781c-46f2-8110-180385d01b58"
-					(reference "#PWR012")
+					(reference "#PWR010")
 					(unit 1)
 				)
@@
 		(dnp no)
 		(fields_autoplaced yes)
-		(property "Reference" "#PWR013"
+		(property "Reference" "#PWR011"
 			(at 193.04 133.35 0)
 			(hide yes)
@@
 			(project "Peculiar"
 				(path "/db27cf5d-1015-467f-a739-ab2eb7f0a1b5/f65afffd-781c-46f2-8110-180385d01b58"
-					(reference "#PWR013")
+					(reference "#PWR011")
 					(unit 1)
 				)
@@
 		(dnp no)
 		(fields_autoplaced yes)
-		(property "Reference" "#PWR09"
+		(property "Reference" "#PWR06"
 			(at 104.14 105.41 0)
 			(hide yes)
@@
 			(project "Peculiar"
 				(path "/db27cf5d-1015-467f-a739-ab2eb7f0a1b5/f65afffd-781c-46f2-8110-180385d01b58"
-					(reference "#PWR09")
+					(reference "#PWR06")
 					(unit 1)
 				)
@@
 		(dnp no)
 		(fields_autoplaced yes)
-		(property "Reference" "#PWR011"
+		(property "Reference" "#PWR012"
 			(at 205.74 87.63 0)
 			(hide yes)
@@
 			(project "Peculiar"
 				(path "/db27cf5d-1015-467f-a739-ab2eb7f0a1b5/f65afffd-781c-46f2-8110-180385d01b58"
-					(reference "#PWR011")
+					(reference "#PWR012")
 					(unit 1)
 				)
@@
 		(in_pos_files yes)
 		(dnp no)
-		(property "Reference" "U3"
+		(property "Reference" "U2"
 			(at 215.9 96.5902 0)
 			(show_name no)
@@
 			(project "Peculiar"
 				(path "/db27cf5d-1015-467f-a739-ab2eb7f0a1b5/f65afffd-781c-46f2-8110-180385d01b58"
-					(reference "U3")
+					(reference "U2")
 					(unit 1)
 				)
@@
 		(dnp no)
 		(fields_autoplaced yes)
-		(property "Reference" "R2"
+		(property "Reference" "R1"
 			(at 157.48 93.9799 0)
 			(show_name no)
@@
 			(project "Peculiar"
 				(path "/db27cf5d-1015-467f-a739-ab2eb7f0a1b5/f65afffd-781c-46f2-8110-180385d01b58"
-					(reference "R2")
+					(reference "R1")
 					(unit 1)
 				)
@@
 		(in_pos_files yes)
 		(dnp no)
-		(property "Reference" "U2"
+		(property "Reference" "U1"
 			(at 177.8 121.9902 0)
 			(show_name no)
@@
 			(project "Peculiar"
 				(path "/db27cf5d-1015-467f-a739-ab2eb7f0a1b5/f65afffd-781c-46f2-8110-180385d01b58"
-					(reference "U2")
+					(reference "U1")
 					(unit 1)
 				)
@@
 		(dnp no)
 		(fields_autoplaced yes)
-		(property "Reference" "R1"
+		(property "Reference" "R3"
 			(at 205.74 69.85 90)
 			(show_name no)
@@
 			(project "Peculiar"
 				(path "/db27cf5d-1015-467f-a739-ab2eb7f0a1b5/f65afffd-781c-46f2-8110-180385d01b58"
-					(reference "R1")
+					(reference "R3")
 					(unit 1)
 				)
@@
 		(dnp no)
 		(fields_autoplaced yes)
-		(property "Reference" "#PWR05"
+		(property "Reference" "#PWR03"
 			(at 78.74 106.68 0)
 			(hide yes)
@@
 			(project "Peculiar"
 				(path "/db27cf5d-1015-467f-a739-ab2eb7f0a1b5/f65afffd-781c-46f2-8110-180385d01b58"
-					(reference "#PWR05")
+					(reference "#PWR03")
 					(unit 1)
 				)
@@
 		(dnp no)
 		(fields_autoplaced yes)
-		(property "Reference" "#PWR06"
+		(property "Reference" "#PWR04"
 			(at 91.44 83.82 0)
 			(hide yes)
@@
 			(project "Peculiar"
 				(path "/db27cf5d-1015-467f-a739-ab2eb7f0a1b5/f65afffd-781c-46f2-8110-180385d01b58"
-					(reference "#PWR06")
+					(reference "#PWR04")
 					(unit 1)
 				)
@@
 		(dnp no)
 		(fields_autoplaced yes)
-		(property "Reference" "C1"
+		(property "Reference" "C2"
 			(at 173.99 93.98 90)
 			(show_name no)
@@
 			(project "Peculiar"
 				(path "/db27cf5d-1015-467f-a739-ab2eb7f0a1b5/f65afffd-781c-46f2-8110-180385d01b58"
-					(reference "C1")
+					(reference "C2")
 					(unit 1)
 				)
@@
 		(dnp no)
 		(fields_autoplaced yes)
-		(property "Reference" "#PWR07"
+		(property "Reference" "#PWR02"
 			(at 78.74 93.98 0)
 			(hide yes)
@@
 			(project "Peculiar"
 				(path "/db27cf5d-1015-467f-a739-ab2eb7f0a1b5/f65afffd-781c-46f2-8110-180385d01b58"
-					(reference "#PWR07")
+					(reference "#PWR02")
 					(unit 1)
 				)
@@
 		(dnp no)
 		(fields_autoplaced yes)
-		(property "Reference" "C2"
+		(property "Reference" "C3"
 			(at 196.85 119.3799 0)
 			(show_name no)
@@
 			(project "Peculiar"
 				(path "/db27cf5d-1015-467f-a739-ab2eb7f0a1b5/f65afffd-781c-46f2-8110-180385d01b58"
-					(reference "C2")
+					(reference "C3")
 					(unit 1)
 				)
@@
 		(dnp no)
 		(fields_autoplaced yes)
-		(property "Reference" "#PWR02"
+		(property "Reference" "#PWR09"
 			(at 167.64 102.87 0)
 			(hide yes)
@@
 			(project "Peculiar"
 				(path "/db27cf5d-1015-467f-a739-ab2eb7f0a1b5/f65afffd-781c-46f2-8110-180385d01b58"
-					(reference "#PWR02")
+					(reference "#PWR09")
 					(unit 1)
 				)
@@
 		(dnp no)
 		(fields_autoplaced yes)
-		(property "Reference" "#PWR04"
+		(property "Reference" "#PWR07"
 			(at 142.24 107.95 0)
 			(hide yes)
@@
 			(project "Peculiar"
 				(path "/db27cf5d-1015-467f-a739-ab2eb7f0a1b5/f65afffd-781c-46f2-8110-180385d01b58"
-					(reference "#PWR04")
+					(reference "#PWR07")
 					(unit 1)
 				)
@@
 		(dnp no)
 		(fields_autoplaced yes)
-		(property "Reference" "#PWR08"
+		(property "Reference" "#PWR05"
 			(at 91.44 96.52 0)
 			(hide yes)
@@
 			(project "Peculiar"
 				(path "/db27cf5d-1015-467f-a739-ab2eb7f0a1b5/f65afffd-781c-46f2-8110-180385d01b58"
-					(reference "#PWR08")
+					(reference "#PWR05")
 					(unit 1)
 				)
@@
 		(dnp no)
 		(fields_autoplaced yes)
-		(property "Reference" "#PWR010"
+		(property "Reference" "#PWR01"
 			(at 66.04 106.68 0)
 			(hide yes)
@@
 			(project "Peculiar"
 				(path "/db27cf5d-1015-467f-a739-ab2eb7f0a1b5/f65afffd-781c-46f2-8110-180385d01b58"
-					(reference "#PWR010")
+					(reference "#PWR01")
 					(unit 1)
 				)
@@
 		(dnp no)
 		(fields_autoplaced yes)
-		(property "Reference" "#PWR01"
+		(property "Reference" "#PWR013"
 			(at 205.74 95.25 0)
 			(hide yes)
@@
 			(project "Peculiar"
 				(path "/db27cf5d-1015-467f-a739-ab2eb7f0a1b5/f65afffd-781c-46f2-8110-180385d01b58"
-					(reference "#PWR01")
+					(reference "#PWR013")
 					(unit 1)
 				)
@@
 		(dnp no)
 		(fields_autoplaced yes)
-		(property "Reference" "R3"
+		(property "Reference" "R2"
 			(at 186.69 107.95 90)
 			(show_name no)
@@
 			(project "Peculiar"
 				(path "/db27cf5d-1015-467f-a739-ab2eb7f0a1b5/f65afffd-781c-46f2-8110-180385d01b58"
-					(reference "R3")
+					(reference "R2")
 					(unit 1)
 				)
@@
 		(dnp no)
 		(fields_autoplaced yes)
-		(property "Reference" "C3"
+		(property "Reference" "C1"
 			(at 146.05 93.9799 0)
 			(show_name no)
@@
 			(project "Peculiar"
 				(path "/db27cf5d-1015-467f-a739-ab2eb7f0a1b5/f65afffd-781c-46f2-8110-180385d01b58"
-					(reference "C3")
+					(reference "C1")
 					(unit 1)
 				)
@@
 		(dnp no)
 		(fields_autoplaced yes)
-		(property "Reference" "#PWR03"
+		(property "Reference" "#PWR08"
 			(at 156.21 119.38 0)
 			(hide yes)
@@
 			(project "Peculiar"
 				(path "/db27cf5d-1015-467f-a739-ab2eb7f0a1b5/f65afffd-781c-46f2-8110-180385d01b58"
-					(reference "#PWR03")
-					(unit 1)
-				)
+					(reference "#PWR08")
+					(unit 1)
+				)
