File: Electronics/Peculiar/Nested simple.kicad_sch (KiCad schematic)
At the start: 12 parts, among them U12 ${SIM.PARAMS}, U13 ${SIM.PARAMS}

Commit message: Create a great design using OPA858 and OPA162
Parts:
- renumbered C14 to C6, CP10 to CP1, CP11 to CP2, CP15 to CP3, CP12 to CP4, R10 to R6, R13 to R7, U12 to U6, U13 to U7
Changed lines of the file:
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@@
 		(dnp no)
 		(fields_autoplaced yes)
-		(property "Reference" "#PWR026"
+		(property "Reference" "#PWR030"
 			(at 86.36 181.61 0)
 			(hide yes)
@@
 			(project "Peculiar"
 				(path "/db27cf5d-1015-467f-a739-ab2eb7f0a1b5/a77c6182-4376-457a-a9e3-921f40aca512"
-					(reference "#PWR026")
+					(reference "#PWR030")
 					(unit 1)
 				)
@@
 		(dnp no)
 		(fields_autoplaced yes)
-		(property "Reference" "#PWR039"
+		(property "Reference" "#PWR041"
 			(at 140.97 119.38 0)
 			(hide yes)
@@
 			(project "Peculiar"
 				(path "/db27cf5d-1015-467f-a739-ab2eb7f0a1b5/a77c6182-4376-457a-a9e3-921f40aca512"
-					(reference "#PWR039")
+					(reference "#PWR041")
 					(unit 1)
 				)
@@
 		(dnp no)
 		(fields_autoplaced yes)
-		(property "Reference" "#PWR036"
+		(property "Reference" "#PWR040"
 			(at 127 120.65 0)
 			(hide yes)
@@
 			(project "Peculiar"
 				(path "/db27cf5d-1015-467f-a739-ab2eb7f0a1b5/a77c6182-4376-457a-a9e3-921f40aca512"
-					(reference "#PWR036")
+					(reference "#PWR040")
 					(unit 1)
 				)
@@
 		(dnp no)
 		(fields_autoplaced yes)
-		(property "Reference" "#PWR037"
+		(property "Reference" "#PWR034"
 			(at 111.76 158.75 0)
 			(hide yes)
@@
 			(project "Peculiar"
 				(path "/db27cf5d-1015-467f-a739-ab2eb7f0a1b5/a77c6182-4376-457a-a9e3-921f40aca512"
-					(reference "#PWR037")
+					(reference "#PWR034")
 					(unit 1)
 				)
@@
 		(dnp no)
 		(fields_autoplaced yes)
-		(property "Reference" "C14"
+		(property "Reference" "C6"
 			(at 130.81 93.9799 0)
 			(show_name no)
@@
 			(project "Peculiar"
 				(path "/db27cf5d-1015-467f-a739-ab2eb7f0a1b5/a77c6182-4376-457a-a9e3-921f40aca512"
-					(reference "C14")
+					(reference "C6")
 					(unit 1)
 				)
@@
 		(dnp no)
 		(fields_autoplaced yes)
-		(property "Reference" "#PWR031"
+		(property "Reference" "#PWR033"
 			(at 101.6 132.08 0)
 			(hide yes)
@@
 			(project "Peculiar"
 				(path "/db27cf5d-1015-467f-a739-ab2eb7f0a1b5/a77c6182-4376-457a-a9e3-921f40aca512"
-					(reference "#PWR031")
+					(reference "#PWR033")
 					(unit 1)
 				)
@@
 		(dnp no)
 		(fields_autoplaced yes)
-		(property "Reference" "#PWR038"
+		(property "Reference" "#PWR035"
 			(at 111.76 171.45 0)
 			(hide yes)
@@
 			(project "Peculiar"
 				(path "/db27cf5d-1015-467f-a739-ab2eb7f0a1b5/a77c6182-4376-457a-a9e3-921f40aca512"
-					(reference "#PWR038")
+					(reference "#PWR035")
 					(unit 1)
 				)
@@
 		(dnp no)
 		(fields_autoplaced yes)
-		(property "Reference" "CP12"
+		(property "Reference" "CP4"
 			(at 158.75 81.28 90)
 			(show_name no)
@@
 			(project "Peculiar"
 				(path "/db27cf5d-1015-467f-a739-ab2eb7f0a1b5/a77c6182-4376-457a-a9e3-921f40aca512"
-					(reference "CP12")
+					(reference "CP4")
 					(unit 1)
 				)
@@
 		(dnp no)
 		(fields_autoplaced yes)
-		(property "Reference" "CP10"
+		(property "Reference" "CP1"
 			(at 105.41 119.3799 0)
 			(show_name no)
@@
 			(project "Peculiar"
 				(path "/db27cf5d-1015-467f-a739-ab2eb7f0a1b5/a77c6182-4376-457a-a9e3-921f40aca512"
-					(reference "CP10")
+					(reference "CP1")
 					(unit 1)
 				)
@@
 		(dnp no)
 		(fields_autoplaced yes)
-		(property "Reference" "#PWR032"
+		(property "Reference" "#PWR036"
 			(at 115.57 119.38 0)
 			(hide yes)
@@
 			(project "Peculiar"
 				(path "/db27cf5d-1015-467f-a739-ab2eb7f0a1b5/a77c6182-4376-457a-a9e3-921f40aca512"
-					(reference "#PWR032")
+					(reference "#PWR036")
 					(unit 1)
 				)
@@
 		(dnp no)
 		(fields_autoplaced yes)
-		(property "Reference" "#PWR035"
+		(property "Reference" "#PWR039"
 			(at 127 113.03 0)
 			(hide yes)
@@
 			(project "Peculiar"
 				(path "/db27cf5d-1015-467f-a739-ab2eb7f0a1b5/a77c6182-4376-457a-a9e3-921f40aca512"
-					(reference "#PWR035")
+					(reference "#PWR039")
 					(unit 1)
 				)
@@
 		(dnp no)
 		(fields_autoplaced yes)
-		(property "Reference" "#PWR052"
+		(property "Reference" "#PWR038"
 			(at 127 69.85 0)
 			(hide yes)
@@
 			(project "Peculiar"
 				(path "/db27cf5d-1015-467f-a739-ab2eb7f0a1b5/a77c6182-4376-457a-a9e3-921f40aca512"
-					(reference "#PWR052")
+					(reference "#PWR038")
 					(unit 1)
 				)
@@
 		(dnp no)
 		(fields_autoplaced yes)
-		(property "Reference" "R13"
+		(property "Reference" "R7"
 			(at 158.75 95.25 90)
 			(show_name no)
@@
 			(project "Peculiar"
 				(path "/db27cf5d-1015-467f-a739-ab2eb7f0a1b5/a77c6182-4376-457a-a9e3-921f40aca512"
-					(reference "R13")
+					(reference "R7")
 					(unit 1)
 				)
@@
 		(dnp no)
 		(fields_autoplaced yes)
-		(property "Reference" "#PWR041"
+		(property "Reference" "#PWR042"
 			(at 152.4 113.03 0)
 			(hide yes)
@@
 			(project "Peculiar"
 				(path "/db27cf5d-1015-467f-a739-ab2eb7f0a1b5/a77c6182-4376-457a-a9e3-921f40aca512"
-					(reference "#PWR041")
+					(reference "#PWR042")
 					(unit 1)
 				)
@@
 		(dnp no)
 		(fields_autoplaced yes)
-		(property "Reference" "#PWR033"
+		(property "Reference" "#PWR031"
 			(at 99.06 168.91 0)
 			(hide yes)
@@
 			(project "Peculiar"
 				(path "/db27cf5d-1015-467f-a739-ab2eb7f0a1b5/a77c6182-4376-457a-a9e3-921f40aca512"
-					(reference "#PWR033")
+					(reference "#PWR031")
 					(unit 1)
 				)
@@
 		(dnp no)
 		(fields_autoplaced yes)
-		(property "Reference" "R10"
+		(property "Reference" "R6"
 			(at 107.95 95.25 90)
 			(show_name no)
@@
 			(project "Peculiar"
 				(path "/db27cf5d-1015-467f-a739-ab2eb7f0a1b5/a77c6182-4376-457a-a9e3-921f40aca512"
-					(reference "R10")
+					(reference "R6")
 					(unit 1)
 				)
@@
 		(dnp no)
 		(fields_autoplaced yes)
-		(property "Reference" "#PWR042"
+		(property "Reference" "#PWR043"
 			(at 152.4 120.65 0)
 			(hide yes)
@@
 			(project "Peculiar"
 				(path "/db27cf5d-1015-467f-a739-ab2eb7f0a1b5/a77c6182-4376-457a-a9e3-921f40aca512"
-					(reference "#PWR042")
+					(reference "#PWR043")
 					(unit 1)
 				)
@@
 		(dnp no)
 		(fields_autoplaced yes)
-		(property "Reference" "#PWR040"
+		(property "Reference" "#PWR037"
 			(at 124.46 180.34 0)
 			(hide yes)
@@
 			(project "Peculiar"
 				(path "/db27cf5d-1015-467f-a739-ab2eb7f0a1b5/a77c6182-4376-457a-a9e3-921f40aca512"
-					(reference "#PWR040")
+					(reference "#PWR037")
 					(unit 1)
 				)
@@
 		(dnp no)
 		(fields_autoplaced yes)
-		(property "Reference" "CP11"
+		(property "Reference" "CP2"
 			(at 107.95 82.55 90)
 			(show_name no)
@@
 			(project "Peculiar"
 				(path "/db27cf5d-1015-467f-a739-ab2eb7f0a1b5/a77c6182-4376-457a-a9e3-921f40aca512"
-					(reference "CP11")
+					(reference "CP2")
 					(unit 1)
 				)
@@
 		(dnp no)
 		(fields_autoplaced yes)
-		(property "Reference" "#PWR034"
+		(property "Reference" "#PWR032"
 			(at 99.06 181.61 0)
 			(hide yes)
@@
 			(project "Peculiar"
 				(path "/db27cf5d-1015-467f-a739-ab2eb7f0a1b5/a77c6182-4376-457a-a9e3-921f40aca512"
-					(reference "#PWR034")
+					(reference "#PWR032")
 					(unit 1)
 				)
@@
 		(in_pos_files yes)
 		(dnp no)
-		(property "Reference" "U12"
+		(property "Reference" "U6"
 			(at 137.16 121.9902 0)
 			(show_name no)
@@
 			(project "Peculiar"
 				(path "/db27cf5d-1015-467f-a739-ab2eb7f0a1b5/a77c6182-4376-457a-a9e3-921f40aca512"
-					(reference "U12")
+					(reference "U6")
 					(unit 1)
 				)
@@
 		(dnp no)
 		(fields_autoplaced yes)
-		(property "Reference" "CP15"
+		(property "Reference" "CP3"
 			(at 143.51 93.9799 0)
 			(show_name no)
@@
 			(project "Peculiar"
 				(path "/db27cf5d-1015-467f-a739-ab2eb7f0a1b5/a77c6182-4376-457a-a9e3-921f40aca512"
-					(reference "CP15")
+					(reference "CP3")
 					(unit 1)
 				)
@@
 		(in_pos_files yes)
 		(dnp no)
-		(property "Reference" "U13"
+		(property "Reference" "U7"
 			(at 162.56 121.9902 0)
 			(show_name no)
@@
 			(project "Peculiar"
 				(path "/db27cf5d-1015-467f-a739-ab2eb7f0a1b5/a77c6182-4376-457a-a9e3-921f40aca512"
-					(reference "U13")
-					(unit 1)
-				)
+					(reference "U7")
+					(unit 1)
+				)
