File: Electronics/Peculiar/Nested.kicad_sch (KiCad schematic)
At the start: 9 parts, among them U6 ${SIM.PARAMS}, U7 ${SIM.PARAMS}, U8 ${SIM.PARAMS}

Commit message: Create a great design using OPA858 and OPA162
Parts:
- renumbered C9 to C5, R7 to R4, R8 to R5, U6 to U3, U7 to U4, U8 to U5
Changed lines of the file:
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@@
 		(dnp no)
 		(fields_autoplaced yes)
-		(property "Reference" "R8"
+		(property "Reference" "R5"
 			(at 101.6 120.65 90)
 			(show_name no)
@@
 			(project "Peculiar"
 				(path "/db27cf5d-1015-467f-a739-ab2eb7f0a1b5/e0f4a773-c283-421c-842f-cbf127c6230d"
-					(reference "R8")
+					(reference "R5")
 					(unit 1)
 				)
@@
 		(dnp no)
 		(fields_autoplaced yes)
-		(property "Reference" "#PWR022"
+		(property "Reference" "#PWR029"
 			(at 114.3 158.75 0)
 			(hide yes)
@@
 			(project "Peculiar"
 				(path "/db27cf5d-1015-467f-a739-ab2eb7f0a1b5/e0f4a773-c283-421c-842f-cbf127c6230d"
-					(reference "#PWR022")
+					(reference "#PWR029")
 					(unit 1)
 				)
@@
 		(dnp no)
 		(fields_autoplaced yes)
-		(property "Reference" "#PWR020"
+		(property "Reference" "#PWR019"
 			(at 63.5 151.13 0)
 			(hide yes)
@@
 			(project "Peculiar"
 				(path "/db27cf5d-1015-467f-a739-ab2eb7f0a1b5/e0f4a773-c283-421c-842f-cbf127c6230d"
-					(reference "#PWR020")
+					(reference "#PWR019")
 					(unit 1)
 				)
@@
 		(dnp no)
 		(fields_autoplaced yes)
-		(property "Reference" "#PWR019"
+		(property "Reference" "#PWR024"
 			(at 85.09 109.22 0)
 			(hide yes)
@@
 			(project "Peculiar"
 				(path "/db27cf5d-1015-467f-a739-ab2eb7f0a1b5/e0f4a773-c283-421c-842f-cbf127c6230d"
-					(reference "#PWR019")
+					(reference "#PWR024")
 					(unit 1)
 				)
@@
 		(dnp no)
 		(fields_autoplaced yes)
-		(property "Reference" "#PWR014"
+		(property "Reference" "#PWR015"
 			(at 46.99 110.49 0)
 			(hide yes)
@@
 			(project "Peculiar"
 				(path "/db27cf5d-1015-467f-a739-ab2eb7f0a1b5/e0f4a773-c283-421c-842f-cbf127c6230d"
-					(reference "#PWR014")
+					(reference "#PWR015")
 					(unit 1)
 				)
@@
 		(dnp no)
 		(fields_autoplaced yes)
-		(property "Reference" "#PWR025"
+		(property "Reference" "#PWR028"
 			(at 114.3 151.13 0)
 			(hide yes)
@@
 			(project "Peculiar"
 				(path "/db27cf5d-1015-467f-a739-ab2eb7f0a1b5/e0f4a773-c283-421c-842f-cbf127c6230d"
-					(reference "#PWR025")
+					(reference "#PWR028")
 					(unit 1)
 				)
@@
 		(dnp no)
 		(fields_autoplaced yes)
-		(property "Reference" "#PWR021"
+		(property "Reference" "#PWR025"
 			(at 88.9 151.13 0)
 			(hide yes)
@@
 			(project "Peculiar"
 				(path "/db27cf5d-1015-467f-a739-ab2eb7f0a1b5/e0f4a773-c283-421c-842f-cbf127c6230d"
-					(reference "#PWR021")
+					(reference "#PWR025")
 					(unit 1)
 				)
@@
 		(dnp no)
 		(fields_autoplaced yes)
-		(property "Reference" "#PWR015"
+		(property "Reference" "#PWR017"
 			(at 59.69 97.79 0)
 			(hide yes)
@@
 			(project "Peculiar"
 				(path "/db27cf5d-1015-467f-a739-ab2eb7f0a1b5/e0f4a773-c283-421c-842f-cbf127c6230d"
-					(reference "#PWR015")
+					(reference "#PWR017")
 					(unit 1)
 				)
@@
 		(dnp no)
 		(fields_autoplaced yes)
-		(property "Reference" "#PWR016"
+		(property "Reference" "#PWR018"
 			(at 59.69 110.49 0)
 			(hide yes)
@@
 			(project "Peculiar"
 				(path "/db27cf5d-1015-467f-a739-ab2eb7f0a1b5/e0f4a773-c283-421c-842f-cbf127c6230d"
-					(reference "#PWR016")
+					(reference "#PWR018")
 					(unit 1)
 				)
@@
 		(dnp no)
 		(fields_autoplaced yes)
-		(property "Reference" "R7"
+		(property "Reference" "R4"
 			(at 91.44 133.35 90)
 			(show_name no)
@@
 			(project "Peculiar"
 				(path "/db27cf5d-1015-467f-a739-ab2eb7f0a1b5/e0f4a773-c283-421c-842f-cbf127c6230d"
-					(reference "R7")
+					(reference "R4")
 					(unit 1)
 				)
@@
 		(dnp no)
 		(fields_autoplaced yes)
-		(property "Reference" "#PWR024"
+		(property "Reference" "#PWR020"
 			(at 63.5 158.75 0)
 			(hide yes)
@@
 			(project "Peculiar"
 				(path "/db27cf5d-1015-467f-a739-ab2eb7f0a1b5/e0f4a773-c283-421c-842f-cbf127c6230d"
-					(reference "#PWR024")
+					(reference "#PWR020")
 					(unit 1)
 				)
@@
 		(dnp no)
 		(fields_autoplaced yes)
-		(property "Reference" "#PWR030"
+		(property "Reference" "#PWR027"
 			(at 102.87 157.48 0)
 			(hide yes)
@@
 			(project "Peculiar"
 				(path "/db27cf5d-1015-467f-a739-ab2eb7f0a1b5/e0f4a773-c283-421c-842f-cbf127c6230d"
-					(reference "#PWR030")
+					(reference "#PWR027")
 					(unit 1)
 				)
@@
 		(dnp no)
 		(fields_autoplaced yes)
-		(property "Reference" "#PWR028"
+		(property "Reference" "#PWR016"
 			(at 52.07 157.48 0)
 			(hide yes)
@@
 			(project "Peculiar"
 				(path "/db27cf5d-1015-467f-a739-ab2eb7f0a1b5/e0f4a773-c283-421c-842f-cbf127c6230d"
-					(reference "#PWR028")
+					(reference "#PWR016")
 					(unit 1)
 				)
@@
 		(dnp no)
 		(fields_autoplaced yes)
-		(property "Reference" "#PWR017"
+		(property "Reference" "#PWR021"
 			(at 72.39 87.63 0)
 			(hide yes)
@@
 			(project "Peculiar"
 				(path "/db27cf5d-1015-467f-a739-ab2eb7f0a1b5/e0f4a773-c283-421c-842f-cbf127c6230d"
-					(reference "#PWR017")
+					(reference "#PWR021")
 					(unit 1)
 				)
@@
 		(dnp no)
 		(fields_autoplaced yes)
-		(property "Reference" "#PWR027"
+		(property "Reference" "#PWR014"
 			(at 38.1 166.37 0)
 			(hide yes)
@@
 			(project "Peculiar"
 				(path "/db27cf5d-1015-467f-a739-ab2eb7f0a1b5/e0f4a773-c283-421c-842f-cbf127c6230d"
-					(reference "#PWR027")
+					(reference "#PWR014")
 					(unit 1)
 				)
@@
 		(in_pos_files yes)
 		(dnp no)
-		(property "Reference" "U7"
+		(property "Reference" "U4"
 			(at 99.06 160.0902 0)
 			(show_name no)
@@
 			(project "Peculiar"
 				(path "/db27cf5d-1015-467f-a739-ab2eb7f0a1b5/e0f4a773-c283-421c-842f-cbf127c6230d"
-					(reference "U7")
+					(reference "U4")
 					(unit 1)
 				)
@@
 		(in_pos_files yes)
 		(dnp no)
-		(property "Reference" "U8"
+		(property "Reference" "U5"
 			(at 124.46 160.0902 0)
 			(show_name no)
@@
 			(project "Peculiar"
 				(path "/db27cf5d-1015-467f-a739-ab2eb7f0a1b5/e0f4a773-c283-421c-842f-cbf127c6230d"
-					(reference "U8")
+					(reference "U5")
 					(unit 1)
 				)
@@
 		(dnp no)
 		(fields_autoplaced yes)
-		(property "Reference" "#PWR029"
+		(property "Reference" "#PWR023"
 			(at 77.47 157.48 0)
 			(hide yes)
@@
 			(project "Peculiar"
 				(path "/db27cf5d-1015-467f-a739-ab2eb7f0a1b5/e0f4a773-c283-421c-842f-cbf127c6230d"
-					(reference "#PWR029")
+					(reference "#PWR023")
 					(unit 1)
 				)
@@
 		(in_pos_files yes)
 		(dnp no)
-		(property "Reference" "U6"
+		(property "Reference" "U3"
 			(at 73.66 160.0902 0)
 			(show_name no)
@@
 			(project "Peculiar"
 				(path "/db27cf5d-1015-467f-a739-ab2eb7f0a1b5/e0f4a773-c283-421c-842f-cbf127c6230d"
-					(reference "U6")
+					(reference "U3")
 					(unit 1)
 				)
@@
 		(dnp no)
 		(fields_autoplaced yes)
-		(property "Reference" "#PWR023"
+		(property "Reference" "#PWR026"
 			(at 88.9 158.75 0)
 			(hide yes)
@@
 			(project "Peculiar"
 				(path "/db27cf5d-1015-467f-a739-ab2eb7f0a1b5/e0f4a773-c283-421c-842f-cbf127c6230d"
-					(reference "#PWR023")
+					(reference "#PWR026")
 					(unit 1)
 				)
@@
 		(dnp no)
 		(fields_autoplaced yes)
-		(property "Reference" "#PWR018"
+		(property "Reference" "#PWR022"
 			(at 72.39 100.33 0)
 			(hide yes)
@@
 			(project "Peculiar"
 				(path "/db27cf5d-1015-467f-a739-ab2eb7f0a1b5/e0f4a773-c283-421c-842f-cbf127c6230d"
-					(reference "#PWR018")
+					(reference "#PWR022")
 					(unit 1)
 				)
@@
 		(dnp no)
 		(fields_autoplaced yes)
-		(property "Reference" "C9"
+		(property "Reference" "C5"
 			(at 41.91 154.9399 0)
 			(show_name no)
@@
 			(project "Peculiar"
 				(path "/db27cf5d-1015-467f-a739-ab2eb7f0a1b5/e0f4a773-c283-421c-842f-cbf127c6230d"
-					(reference "C9")
-					(unit 1)
-				)
+					(reference "C5")
+					(unit 1)
+				)
