File: Electronics/Peculiar/Peculiar.kicad_sch (KiCad schematic)
At the start: 0 parts

Commit message: Create a great design using OPA858 and OPA162
Other:
- added sheet OPA858 and OPA162 (OPA858 and OPA162.kicad_sch)
Changed lines of the file:
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@@
 	(paper "A4")
 	(sheet
-		(at 166.37 143.51)
-		(size 22.86 11.43)
+		(at 50.8 25.4)
+		(size 12.7 12.7)
 		(exclude_from_sim yes)
 		(in_bom yes)
@@
 		)
 		(property "Sheetname" "Three Op Amps"
-			(at 166.37 142.7984 0)
+			(at 50.8 24.6884 0)
 			(show_name no)
 			(do_not_autoplace no)
@@
 		)
 		(property "Sheetfile" "Three Op Amps.kicad_sch"
-			(at 166.37 155.5246 0)
+			(at 50.8 38.6846 0)
 			(show_name no)
 			(do_not_autoplace no)
@@
 	)
 	(sheet
-		(at 127 111.76)
-		(size 29.21 21.59)
+		(at 25.4 101.6)
+		(size 12.7 12.7)
+		(exclude_from_sim yes)
+		(in_bom yes)
+		(on_board yes)
+		(dnp no)
+		(fields_autoplaced yes)
+		(stroke
+			(width 0.1524)
+			(type solid)
+		)
+		(fill
+			(color 0 0 0 0)
+		)
+		(property "Sheetname" "OPA858"
+			(at 25.4 100.8884 0)
+			(show_name no)
+			(do_not_autoplace no)
+			(effects
+				(font
+					(size 1.27 1.27)
+				)
+				(justify left bottom)
+			)
+		)
+		(property "Sheetfile" "OPA858.kicad_sch"
+			(at 25.4 114.8846 0)
+			(show_name no)
+			(do_not_autoplace no)
+			(effects
+				(font
+					(size 1.27 1.27)
+				)
+				(justify left top)
+			)
+		)
+		(instances
+			(project "Peculiar"
+				(path "/db27cf5d-1015-467f-a739-ab2eb7f0a1b5"
+					(page "5")
+				)
+			)
+		)
+	)
+	(sheet
+		(at 25.4 127)
+		(size 12.7 12.7)
+		(exclude_from_sim yes)
+		(in_bom yes)
+		(on_board yes)
+		(dnp no)
+		(fields_autoplaced yes)
+		(stroke
+			(width 0.1524)
+			(type solid)
+		)
+		(fill
+			(color 0 0 0 0)
+		)
+		(property "Sheetname" "LMC606"
+			(at 25.4 126.2884 0)
+			(show_name no)
+			(do_not_autoplace no)
+			(effects
+				(font
+					(size 1.27 1.27)
+				)
+				(justify left bottom)
+			)
+		)
+		(property "Sheetfile" "LMC606.kicad_sch"
+			(at 25.4 140.2846 0)
+			(show_name no)
+			(do_not_autoplace no)
+			(effects
+				(font
+					(size 1.27 1.27)
+				)
+				(justify left top)
+			)
+		)
+		(instances
+			(project "Peculiar"
+				(path "/db27cf5d-1015-467f-a739-ab2eb7f0a1b5"
+					(page "6")
+				)
+			)
+		)
+	)
+	(sheet
+		(at 25.4 76.2)
+		(size 12.7 12.7)
+		(exclude_from_sim yes)
+		(in_bom yes)
+		(on_board yes)
+		(dnp no)
+		(fields_autoplaced yes)
+		(stroke
+			(width 0.1524)
+			(type solid)
+		)
+		(fill
+			(color 0 0 0 0)
+		)
+		(property "Sheetname" "Nested simple"
+			(at 25.4 75.4884 0)
+			(show_name no)
+			(do_not_autoplace no)
+			(effects
+				(font
+					(size 1.27 1.27)
+				)
+				(justify left bottom)
+			)
+		)
+		(property "Sheetfile" "Nested simple.kicad_sch"
+			(at 25.4 89.4846 0)
+			(show_name no)
+			(do_not_autoplace no)
+			(effects
+				(font
+					(size 1.27 1.27)
+				)
+				(justify left top)
+			)
+		)
+		(instances
+			(project "Peculiar"
+				(path "/db27cf5d-1015-467f-a739-ab2eb7f0a1b5"
+					(page "4")
+				)
+			)
+		)
+	)
+	(sheet
+		(at 25.4 152.4)
+		(size 12.7 12.7)
 		(exclude_from_sim no)
 		(in_bom yes)
@@
 			(color 0 0 0 0)
 		)
-		(property "Sheetname" "OPA858"
-			(at 127 111.0484 0)
-			(show_name no)
-			(do_not_autoplace no)
-			(effects
-				(font
-					(size 1.27 1.27)
-				)
-				(justify left bottom)
-			)
-		)
-		(property "Sheetfile" "OPA858.kicad_sch"
-			(at 127 133.9346 0)
-			(show_name no)
-			(do_not_autoplace no)
-			(effects
-				(font
-					(size 1.27 1.27)
-				)
-				(justify left top)
-			)
-		)
-		(instances
-			(project "Peculiar"
-				(path "/db27cf5d-1015-467f-a739-ab2eb7f0a1b5"
-					(page "5")
-				)
-			)
-		)
-	)
-	(sheet
-		(at 83.82 148.59)
-		(size 30.48 12.7)
-		(exclude_from_sim yes)
-		(in_bom yes)
-		(on_board yes)
-		(dnp no)
-		(fields_autoplaced yes)
-		(stroke
-			(width 0.1524)
-			(type solid)
-		)
-		(fill
-			(color 0 0 0 0)
-		)
-		(property "Sheetname" "LMC606"
-			(at 83.82 147.8784 0)
-			(show_name no)
-			(do_not_autoplace no)
-			(effects
-				(font
-					(size 1.27 1.27)
-				)
-				(justify left bottom)
-			)
-		)
-		(property "Sheetfile" "LMC606.kicad_sch"
-			(at 83.82 161.8746 0)
-			(show_name no)
-			(do_not_autoplace no)
-			(effects
-				(font
-					(size 1.27 1.27)
-				)
-				(justify left top)
-			)
-		)
-		(instances
-			(project "Peculiar"
-				(path "/db27cf5d-1015-467f-a739-ab2eb7f0a1b5"
-					(page "6")
-				)
-			)
-		)
-	)
-	(sheet
-		(at 78.74 113.03)
-		(size 25.4 24.13)
-		(exclude_from_sim yes)
-		(in_bom yes)
-		(on_board yes)
-		(dnp no)
-		(fields_autoplaced yes)
-		(stroke
-			(width 0.1524)
-			(type solid)
-		)
-		(fill
-			(color 0 0 0 0)
-		)
-		(property "Sheetname" "Nested simple"
-			(at 78.74 112.3184 0)
-			(show_name no)
-			(do_not_autoplace no)
-			(effects
-				(font
-					(size 1.27 1.27)
-				)
-				(justify left bottom)
-			)
-		)
-		(property "Sheetfile" "Nested simple.kicad_sch"
-			(at 78.74 137.7446 0)
-			(show_name no)
-			(do_not_autoplace no)
-			(effects
-				(font
-					(size 1.27 1.27)
-				)
-				(justify left top)
-			)
-		)
-		(instances
-			(project "Peculiar"
-				(path "/db27cf5d-1015-467f-a739-ab2eb7f0a1b5"
-					(page "4")
-				)
-			)
-		)
-	)
-	(sheet
-		(at 33.02 111.76)
-		(size 21.59 24.13)
+		(property "Sheetname" "OPA858 and OPA162"
+			(at 25.4 151.6884 0)
+			(show_name no)
+			(do_not_autoplace no)
+			(effects
+				(font
+					(size 1.27 1.27)
+				)
+				(justify left bottom)
+			)
+		)
+		(property "Sheetfile" "OPA858 and OPA162.kicad_sch"
+			(at 25.4 165.6846 0)
+			(show_name no)
+			(do_not_autoplace no)
+			(effects
+				(font
+					(size 1.27 1.27)
+				)
+				(justify left top)
+			)
+		)
+		(instances
+			(project "Peculiar"
+				(path "/db27cf5d-1015-467f-a739-ab2eb7f0a1b5"
+					(page "7")
+				)
+			)
+		)
+	)
+	(sheet
+		(at 25.4 50.8)
+		(size 12.7 12.7)
 		(exclude_from_sim yes)
 		(in_bom yes)
@@
 		)
 		(property "Sheetname" "Nested"
-			(at 33.02 111.0484 0)
+			(at 25.4 50.0884 0)
 			(show_name no)
 			(do_not_autoplace no)
@@
 		)
 		(property "Sheetfile" "Nested.kicad_sch"
-			(at 33.02 136.4746 0)
+			(at 25.4 64.0846 0)
 			(show_name no)
 			(do_not_autoplace no)
@@
 		)
 		(property "Field2" ""
-			(at 33.02 111.76 0)
+			(at 25.4 50.8 0)
 			(hide yes)
 			(show_name no)
@@
 	)
 	(sheet
-		(at 33.02 69.85)
-		(size 27.94 22.86)
+		(at 25.4 25.4)
+		(size 12.7 12.7)
 		(exclude_from_sim yes)
 		(in_bom yes)
@@
 		)
 		(property "Sheetname" "From OPA380"
-			(at 33.02 69.1384 0)
+			(at 25.4 24.6884 0)
 			(show_name no)
 			(do_not_autoplace no)
@@
 		)
 		(property "Sheetfile" "From OPA380.kicad_sch"
-			(at 33.02 93.2946 0)
-			(show_name no)
-			(do_not_autoplace no)
+			(at 25.4 38.6846 0)
+			(show_name no)
+			(do_not_autoplace no)
