File: Electronics/Peculiar/Three Op Amps.kicad_sch (KiCad schematic)
At the start: 12 parts, among them U15 ${SIM.PARAMS}, U18 ${SIM.PARAMS}

Commit message: Create some other simulations
Parts:
- removed C15: 1n, symbol Device:C
- removed CP13: 10n, symbol Device:C
- removed CP14, CP17: 100f, symbol Device:C
- removed CP16: 100p, symbol Device:C
- removed I4: ISIN, symbol Simulation_SPICE:ISIN
- removed R11: 10M, symbol Device:R
- removed R14: 900, symbol Device:R
- removed U15, U18: ${SIM.PARAMS}, symbol Simulation_SPICE:OPAMP
- removed V7, V8: 5V, symbol Simulation_SPICE:VDC
- added C18: 1n, symbol Device:C
- added CP26: 10n, symbol Device:C
- added CP27, CP29: 100f, symbol Device:C
- added CP28: 100p, symbol Device:C
- added I7: ISIN, symbol Simulation_SPICE:ISIN
- added R18: 10M, symbol Device:R
- added R19: 900, symbol Device:R
- added U22, U23, U24: ${SIM.PARAMS}, symbol Simulation_SPICE:OPAMP
- added V13, V14: 5V, symbol Simulation_SPICE:VDC
Connections:
- net +5V: now also U22.3 (V+), U23.3 (V+), U24.3 (V+), V13.1
- net -5V: now also U22.4 (V-), U23.4 (V-), U24.4 (V-), V14.2
- net 0: now also C18.2, CP26.2, CP28.2, I7.2, U22.1 (+), U23.1 (+), U24.1 (+), V13.2, V14.1
- net VIN: now also CP26.1, CP27.1, I7.1, R18.1, U22.2 (-)
- net VOUT: now also CP29.2, R19.2, U24.5
- new net: C18.1, CP27.2, CP28.1, CP29.1, R18.2, R19.1
- new net: U22.5, U23.2 (-)
- new net: U23.5, U24.2 (-)

Commit message: Separate two and three OPA858 designs
Parts:
- removed C18: 1n, symbol Device:C
- removed CP26: 10n, symbol Device:C
- removed CP27, CP29: 100f, symbol Device:C
- removed CP28: 100p, symbol Device:C
- removed I7: ISIN, symbol Simulation_SPICE:ISIN
- removed U23, U24: ${SIM.PARAMS}, symbol Simulation_SPICE:OPAMP
- removed V13, V14: 5V, symbol Simulation_SPICE:VDC
- added C17: 1n, symbol Device:C
- added CP22: 100n, symbol Device:C
- added CP23: 200f, symbol Device:C
- added CP24: 10p, symbol Device:C
- added CP25: 1p, symbol Device:C
- added I6: ISIN, symbol Simulation_SPICE:ISIN
- added R17: 10M, symbol Device:R
- added U20, U21: ${SIM.PARAMS}, symbol Simulation_SPICE:OPAMP
- added V11, V12: 5V, symbol Simulation_SPICE:VDC
- R18: value 10M -> 100k
- R19: value 900 -> 2000
Connections:
- net +5V: now also U20.3 (V+), U21.3 (V+), V11.1
- net -5V: now also U20.4 (V-), U21.4 (V-), V12.2
- net 0: now also C17.2, CP22.2, CP24.2, I6.2, U20.1 (+), U21.1 (+), V11.2, V12.1
- net VIN: now also CP22.1, CP23.1, I6.1, R17.1, U20.2 (-); no longer R18.1, U22.2 (-)
- net VOUT: now also U22.5, CP25.2
- net at R18.2, R19.1: now also C17.1, CP23.2, CP24.1, CP25.1
- new net: U20.5, U21.2 (-)
- new net: R17.2, R18.1
- new net: U21.5, U22.2 (-)

Commit message: Create a great design using OPA858 and OPA162
Parts:
- renumbered C17 to C10, CP22 to CP20, CP23 to CP21, CP24 to CP22, CP25 to CP23, I6 to I7, R17 to R15, R18 to R16, R19 to R17, U20 to U15, U21 to U16, U22 to U17, V11 to V13, V12 to V14
