File: Electronics/TIA/OPA858 Stage.kicad_sch (KiCad schematic)
At the start: 5 parts, among them U5 ${SIM.PARAMS}

Commit message: Mess around with the simulation
Parts:
- R15: renamed from R11; value 47 -> 10
Changed lines of the file:
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@@
+					(unit 1)
+				)
+				(path "/71573f97-d585-4d55-ac00-8cb3ed311569/7393f255-b863-4c1d-9342-5a39256b0530/6574afd4-ee93-4d54-b19b-de84322b8512"
+					(reference "LP5")
 					(unit 1)
 				)
 				(path "/71573f97-d585-4d55-ac00-8cb3ed311569/7393f255-b863-4c1d-9342-5a39256b0530/7522ab81-de0c-4e4a-866e-c0efc6c9785b"
 					(reference "LP4")
-					(unit 1)
-				)
-				(path "/71573f97-d585-4d55-ac00-8cb3ed311569/7393f255-b863-4c1d-9342-5a39256b0530/a6d32514-4da2-4918-8e0e-712121b4b2e2"
-					(reference "LP5")
 					(unit 1)
 				)
@@
 		(dnp no)
 		(fields_autoplaced yes)
-		(property "Reference" "#PWR032"
+		(property "Reference" "#PWR037"
 			(at 127 82.55 0)
 			(effects
@@
 			(project "TIA"
 				(path "/71573f97-d585-4d55-ac00-8cb3ed311569/7393f255-b863-4c1d-9342-5a39256b0530/3ecb7f7a-1c03-4eaf-a122-686264238360"
-					(reference "#PWR032")
-					(unit 1)
-				)
-				(path "/71573f97-d585-4d55-ac00-8cb3ed311569/7393f255-b863-4c1d-9342-5a39256b0530/7522ab81-de0c-4e4a-866e-c0efc6c9785b"
-					(reference "#PWR036")
-					(unit 1)
-				)
-				(path "/71573f97-d585-4d55-ac00-8cb3ed311569/7393f255-b863-4c1d-9342-5a39256b0530/a6d32514-4da2-4918-8e0e-712121b4b2e2"
-					(reference "#PWR040")
+					(reference "#PWR037")
+					(unit 1)
+				)
+				(path "/71573f97-d585-4d55-ac00-8cb3ed311569/7393f255-b863-4c1d-9342-5a39256b0530/6574afd4-ee93-4d54-b19b-de84322b8512"
+					(reference "#PWR027")
+					(unit 1)
+				)
+				(path "/71573f97-d585-4d55-ac00-8cb3ed311569/7393f255-b863-4c1d-9342-5a39256b0530/7522ab81-de0c-4e4a-866e-c0efc6c9785b"
+					(reference "#PWR041")
 					(unit 1)
 				)
@@
 					(unit 1)
 				)
+				(path "/71573f97-d585-4d55-ac00-8cb3ed311569/7393f255-b863-4c1d-9342-5a39256b0530/6574afd4-ee93-4d54-b19b-de84322b8512"
+					(reference "U7")
+					(unit 1)
+				)
 				(path "/71573f97-d585-4d55-ac00-8cb3ed311569/7393f255-b863-4c1d-9342-5a39256b0530/7522ab81-de0c-4e4a-866e-c0efc6c9785b"
 					(reference "U6")
-					(unit 1)
-				)
-				(path "/71573f97-d585-4d55-ac00-8cb3ed311569/7393f255-b863-4c1d-9342-5a39256b0530/a6d32514-4da2-4918-8e0e-712121b4b2e2"
-					(reference "U7")
 					(unit 1)
 				)
@@
 		(dnp no)
 		(fields_autoplaced yes)
-		(property "Reference" "#PWR031"
+		(property "Reference" "#PWR036"
 			(at 127 74.93 0)
 			(effects
@@
 			(project "TIA"
 				(path "/71573f97-d585-4d55-ac00-8cb3ed311569/7393f255-b863-4c1d-9342-5a39256b0530/3ecb7f7a-1c03-4eaf-a122-686264238360"
-					(reference "#PWR031")
-					(unit 1)
-				)
-				(path "/71573f97-d585-4d55-ac00-8cb3ed311569/7393f255-b863-4c1d-9342-5a39256b0530/7522ab81-de0c-4e4a-866e-c0efc6c9785b"
-					(reference "#PWR035")
-					(unit 1)
-				)
-				(path "/71573f97-d585-4d55-ac00-8cb3ed311569/7393f255-b863-4c1d-9342-5a39256b0530/a6d32514-4da2-4918-8e0e-712121b4b2e2"
-					(reference "#PWR039")
+					(reference "#PWR036")
+					(unit 1)
+				)
+				(path "/71573f97-d585-4d55-ac00-8cb3ed311569/7393f255-b863-4c1d-9342-5a39256b0530/6574afd4-ee93-4d54-b19b-de84322b8512"
+					(reference "#PWR024")
+					(unit 1)
+				)
+				(path "/71573f97-d585-4d55-ac00-8cb3ed311569/7393f255-b863-4c1d-9342-5a39256b0530/7522ab81-de0c-4e4a-866e-c0efc6c9785b"
+					(reference "#PWR040")
 					(unit 1)
 				)
@@
 		(dnp no)
 		(fields_autoplaced yes)
-		(property "Reference" "#PWR030"
+		(property "Reference" "#PWR035"
 			(at 115.57 81.28 0)
 			(effects
@@
 			(project "TIA"
 				(path "/71573f97-d585-4d55-ac00-8cb3ed311569/7393f255-b863-4c1d-9342-5a39256b0530/3ecb7f7a-1c03-4eaf-a122-686264238360"
-					(reference "#PWR030")
-					(unit 1)
-				)
-				(path "/71573f97-d585-4d55-ac00-8cb3ed311569/7393f255-b863-4c1d-9342-5a39256b0530/7522ab81-de0c-4e4a-866e-c0efc6c9785b"
-					(reference "#PWR034")
-					(unit 1)
-				)
-				(path "/71573f97-d585-4d55-ac00-8cb3ed311569/7393f255-b863-4c1d-9342-5a39256b0530/a6d32514-4da2-4918-8e0e-712121b4b2e2"
-					(reference "#PWR038")
+					(reference "#PWR035")
+					(unit 1)
+				)
+				(path "/71573f97-d585-4d55-ac00-8cb3ed311569/7393f255-b863-4c1d-9342-5a39256b0530/6574afd4-ee93-4d54-b19b-de84322b8512"
+					(reference "#PWR023")
+					(unit 1)
+				)
+				(path "/71573f97-d585-4d55-ac00-8cb3ed311569/7393f255-b863-4c1d-9342-5a39256b0530/7522ab81-de0c-4e4a-866e-c0efc6c9785b"
+					(reference "#PWR039")
 					(unit 1)
 				)
@@
 		(dnp no)
 		(fields_autoplaced yes)
-		(property "Reference" "#PWR033"
+		(property "Reference" "#PWR038"
 			(at 177.8 93.98 0)
 			(effects
@@
 			(project "TIA"
 				(path "/71573f97-d585-4d55-ac00-8cb3ed311569/7393f255-b863-4c1d-9342-5a39256b0530/3ecb7f7a-1c03-4eaf-a122-686264238360"
-					(reference "#PWR033")
-					(unit 1)
-				)
-				(path "/71573f97-d585-4d55-ac00-8cb3ed311569/7393f255-b863-4c1d-9342-5a39256b0530/7522ab81-de0c-4e4a-866e-c0efc6c9785b"
-					(reference "#PWR037")
-					(unit 1)
-				)
-				(path "/71573f97-d585-4d55-ac00-8cb3ed311569/7393f255-b863-4c1d-9342-5a39256b0530/a6d32514-4da2-4918-8e0e-712121b4b2e2"
-					(reference "#PWR041")
+					(reference "#PWR038")
+					(unit 1)
+				)
+				(path "/71573f97-d585-4d55-ac00-8cb3ed311569/7393f255-b863-4c1d-9342-5a39256b0530/6574afd4-ee93-4d54-b19b-de84322b8512"
+					(reference "#PWR028")
+					(unit 1)
+				)
+				(path "/71573f97-d585-4d55-ac00-8cb3ed311569/7393f255-b863-4c1d-9342-5a39256b0530/7522ab81-de0c-4e4a-866e-c0efc6c9785b"
+					(reference "#PWR042")
 					(unit 1)
 				)
@@
 					(unit 1)
 				)
+				(path "/71573f97-d585-4d55-ac00-8cb3ed311569/7393f255-b863-4c1d-9342-5a39256b0530/6574afd4-ee93-4d54-b19b-de84322b8512"
+					(reference "RP4")
+					(unit 1)
+				)
 				(path "/71573f97-d585-4d55-ac00-8cb3ed311569/7393f255-b863-4c1d-9342-5a39256b0530/7522ab81-de0c-4e4a-866e-c0efc6c9785b"
 					(reference "RP3")
-					(unit 1)
-				)
-				(path "/71573f97-d585-4d55-ac00-8cb3ed311569/7393f255-b863-4c1d-9342-5a39256b0530/a6d32514-4da2-4918-8e0e-712121b4b2e2"
-					(reference "RP4")
 					(unit 1)
 				)
@@
 		(dnp no)
 		(fields_autoplaced yes)
-		(property "Reference" "R11"
+		(property "Reference" "R15"
 			(at 146.05 69.85 90)
 			(effects
@@
 			)
 		)
-		(property "Value" "47"
+		(property "Value" "10"
 			(at 146.05 72.39 90)
 			(effects
@@
 			(project "TIA"
 				(path "/71573f97-d585-4d55-ac00-8cb3ed311569/7393f255-b863-4c1d-9342-5a39256b0530/3ecb7f7a-1c03-4eaf-a122-686264238360"
-					(reference "R11")
-					(unit 1)
-				)
-				(path "/71573f97-d585-4d55-ac00-8cb3ed311569/7393f255-b863-4c1d-9342-5a39256b0530/7522ab81-de0c-4e4a-866e-c0efc6c9785b"
-					(reference "R12")
-					(unit 1)
-				)
-				(path "/71573f97-d585-4d55-ac00-8cb3ed311569/7393f255-b863-4c1d-9342-5a39256b0530/a6d32514-4da2-4918-8e0e-712121b4b2e2"
-					(reference "R13")
+					(reference "R15")
+					(unit 1)
+				)
+				(path "/71573f97-d585-4d55-ac00-8cb3ed311569/7393f255-b863-4c1d-9342-5a39256b0530/6574afd4-ee93-4d54-b19b-de84322b8512"
+					(reference "R8")
+					(unit 1)
+				)
+				(path "/71573f97-d585-4d55-ac00-8cb3ed311569/7393f255-b863-4c1d-9342-5a39256b0530/7522ab81-de0c-4e4a-866e-c0efc6c9785b"
+					(reference "R16")
 					(unit 1)
 				)
@@
 					(unit 1)
 				)
+				(path "/71573f97-d585-4d55-ac00-8cb3ed311569/7393f255-b863-4c1d-9342-5a39256b0530/6574afd4-ee93-4d54-b19b-de84322b8512"
+					(reference "CP5")
+					(unit 1)
+				)
 				(path "/71573f97-d585-4d55-ac00-8cb3ed311569/7393f255-b863-4c1d-9342-5a39256b0530/7522ab81-de0c-4e4a-866e-c0efc6c9785b"
 					(reference "CP4")
 					(unit 1)
 				)
-				(path "/71573f97-d585-4d55-ac00-8cb3ed311569/7393f255-b863-4c1d-9342-5a39256b0530/a6d32514-4da2-4918-8e0e-712121b4b2e2"
-					(reference "CP5")
-					(unit 1)
-				)
