File: Electronics/TIA/RS8751.kicad_sch (KiCad schematic)
At the start: 16 parts

Commit message: Simulate a 1G TIA gain again
Parts:
- C5: value 1n -> 100n
- R9: value 10M -> 1G
Other:
- added sheet RS8751 Stage3 (page 10)1 (OPA858 Stage.kicad_sch)
Changed lines of the file:
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@@
-	(wire
-		(pts
-			(xy 203.2 90.17) (xy 203.2 139.7)
-		)
-		(stroke
-			(width 0)
-			(type default)
-		)
-	)
 	(wire
 		(pts
@@
 	(wire
 		(pts
+			(xy 203.2 90.17) (xy 203.2 132.08)
+		)
+		(stroke
+			(width 0)
+			(type default)
+		)
+	)
+	(wire
+		(pts
 			(xy 116.84 63.5) (xy 114.3 63.5)
 		)
@@
 	(wire
 		(pts
+			(xy 203.2 132.08) (xy 208.28 132.08)
+		)
+		(stroke
+			(width 0)
+			(type default)
+		)
+	)
+	(wire
+		(pts
 			(xy 88.9 76.2) (xy 101.6 76.2)
 		)
@@
 	(wire
 		(pts
+			(xy 208.28 132.08) (xy 208.28 139.7)
+		)
+		(stroke
+			(width 0)
+			(type default)
+		)
+	)
+	(wire
+		(pts
 			(xy 101.6 78.74) (xy 101.6 76.2)
 		)
@@
 	(wire
 		(pts
-			(xy 190.5 139.7) (xy 203.2 139.7)
+			(xy 190.5 139.7) (xy 193.04 139.7)
 		)
 		(stroke
@@
 		(pts
 			(xy 25.4 38.1) (xy 25.4 49.53)
+		)
+		(stroke
+			(width 0)
+			(type default)
+		)
+	)
+	(wire
+		(pts
+			(xy 205.74 139.7) (xy 208.28 139.7)
 		)
 		(stroke
@@
 			)
 		)
-		(property "Value" "1n"
+		(property "Value" "100n"
 			(at 156.21 71.1199 0)
 			(effects
@@
 			)
 		)
-		(property "Value" "10M"
+		(property "Value" "1G"
 			(at 120.65 72.39 90)
 			(effects
@@
 				)
 			)
+		)
+	)
+	(sheet
+		(at 193.04 137.16)
+		(size 12.7 5.08)
+		(exclude_from_sim no)
+		(in_bom yes)
+		(on_board yes)
+		(dnp no)
+		(fields_autoplaced yes)
+		(stroke
+			(width 0.1524)
+			(type solid)
+		)
+		(fill
+			(color 0 0 0 0.0000)
+		)
+		(property "Sheetname" "RS8751 Stage3 (page 10)1"
+			(at 193.04 136.4484 0)
+			(effects
+				(font
+					(size 1.27 1.27)
+				)
+				(justify left bottom)
+			)
+		)
+		(property "Sheetfile" "OPA858 Stage.kicad_sch"
+			(at 193.04 142.8246 0)
+			(effects
+				(font
+					(size 1.27 1.27)
+				)
+				(justify left top)
+				(hide yes)
+			)
+		)
+		(pin "IN" input
+			(at 193.04 139.7 180)
+			(effects
+				(font
+					(size 1.27 1.27)
+				)
+				(justify left)
+			)
+		)
+		(pin "OUT" input
+			(at 205.74 139.7 0)
+			(effects
+				(font
+					(size 1.27 1.27)
+				)
+				(justify right)
+			)
+		)
+		(instances
+			(project "TIA"
+				(path "/71573f97-d585-4d55-ac00-8cb3ed311569/447ab444-b820-479d-9c03-ff04d3523599"
+					(page "11")
+				)
+			)

Commit message: Experiment with stabilizing capacitor
Parts:
- C4: value 10n -> 1u
- C5: value 100n -> 10n
- R9: value 1G -> 100M
Changed lines of the file:
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@@
 			)
 		)
-		(property "Value" "100n"
+		(property "Value" "10n"
 			(at 156.21 71.1199 0)
 			(effects
@@
 			)
 		)
-		(property "Value" "10n"
+		(property "Value" "1u"
 			(at 105.41 83.8199 0)
 			(effects
@@
 			)
 		)
-		(property "Value" "1G"
+		(property "Value" "100M"
 			(at 120.65 72.39 90)
 			(effects
