File: Electronics/TIA/TLV906.kicad_sch (KiCad schematic)
At the start: 17 parts, among them U1 ${SIM.PARAMS}, U2 ${SIM.PARAMS}, U3 ${SIM.PARAMS}, U4 ${SIM.PARAMS}

Commit message: Play with the TLV9061 simulation
Parts:
- C1: value 1p -> 10n
Changed lines of the file:
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@@
 			)
 		)
-		(property "Value" "1p"
+		(property "Value" "10n"
 			(at 85.09 92.7099 0)
 			(effects
