File: Electronics/Decoupling capacitors/Decoupling capacitors.kicad_sch (KiCad schematic)
At the start: 35 parts

Commit message: Test more realistic decoupling capacitor values
Parts:
- removed C7, C8: 10u, symbol Device:C
- removed L7, L8: 633.26p, symbol Device:L
- removed R11, R12: 0.006, symbol Device:R
- added C10: 100n, symbol Device:C
- added L10: 281.45p, symbol Device:L
- added R14: 0.02, symbol Device:R
- C6: value 10u -> 100n
- L6: value 633.26p -> 281.45p
- R10: value 0.006 -> 0.02
Connections:
- net 0: now also R14.2
- net OUT4: now also C10.1
- new net: L10.2, R14.1
- new net: C10.2, L10.1
